File: hw/esp32buscam_01.sch (EAGLE design)
At the start: 51 parts, among them IC11 MCP1703DB, IC12 MCP1703DB, IC2 MCP1703DB, K1 68712414522, Q1 IRLML2244, Q4 IRLML2244, U1 ESP32-S2-MINI-1, U2 FLASH, U3 ESP-PSRAM64, X1 JTAG, X2 PROG

Commit message: first 100% layout
Parts:
- removed C1, C5, C6, C7, C9: (no value), rcl:C-EUC0603
- removed GPS: BUS, con-amp-micromatch:MICROMATCH-6SMD
- removed IC11, IC12: MCP1703DB, linear:MCP1703DB
- removed LED_B: G, led:LEDCHIPLED_0805
- removed Q3: (no value), crystal:CRYSTALTC26V
- removed R17, R19, R21, R5: (no value), rcl:R-EU_R0603
- removed RESET: (no value), Ergaenzung:TASTER-9314_SMD
- removed U2: FLASH, esp32s2mini:S25FL127SABMFI103
- removed U3: ESP-PSRAM64, esp32s2mini:S25FL127SABMFI103
- added BUS: BUS, con-amp-micromatch:MICROMATCH-6SMD
- added D1, D2, D3: (no value), diode:DIODE-MINIMELF
- added IC1, IC3: MCP1703SOT-89, bytewerk-vreg:MCP1703SOT-89
- added LED1, LED2: (no value), led:LED5MM
- added LED_DBG: G, led:LEDCHIPLED_0805
- added PAD1, PAD2, PAD3, PAD4, PAD5, PAD6: (no value), wirepad:1,6/0,9
- added Q2: IRLML2244, User-Submitted:MOSFET-PCHANNELIRLML2244
- added SJ1, SJ3, SJ4, SJ5: (no value), jumper:SJ
- BOOT: device Ergaenzung:TASTER-9314_SMD -> jumper:SJ
- IC2: value MCP1703DB -> MCP1703SOT-89; device linear:MCP1703DB -> bytewerk-vreg:MCP1703SOT-89
- R2, R3, R4: device rcl:R-EU_R0603 -> rcl:R-EU_R0402
Connections:
- removed net CAM_HREF: U1.IO3
- removed net CAM_PWDN: K1.17, R17.1
- removed net ESP_CS1: R2.1, U3.!CS
- removed net ESP_CS2: R5.1, U2.!CS
- removed net ESP_TDI(: U1.IO41
- removed net MTDO: R21.2
- removed net N$21: LED_B.A, R21.1
- removed net N$6: U1.IO1
- removed net SD_CMD: R40.2, SDCARD.CMD
- removed net SD_D0: R38.2, SDCARD.DATA0
- removed net SD_D3: R43.2, SDCARD.CD/DATA3
- removed net SPICLK: U2.CLK, U3.CLK
- removed net SPID: U2.SI/IO0, U3.SI/IO0
- removed net SPIHD: U2.!HOLD/IO3, U3.!HOLD/IO3
- removed net SPIQ: U2.SO/IO1, U3.SO/IO1
- removed net SPIWP: U2.!WP/IO2, U3.!WP/IO2
- removed net SPI_MISO: GPS-1.S
- removed net SPI_MOSI: GPS-4.S
- removed net SPI_RESET: GPS-5.S
- removed net SPI_SCK: GPS-3.S
- removed net UBUS: GPS-2.S
- removed net USB_ID: USB.4
- removed net VBAT: C3.1, IC2.VI
- new net BUS_MISO_INT: BUS-1.S, U1.IO45
- new net BUS_MOSI_SDA: BUS-4.S, U1.IO9
- new net BUS_RESET: BUS-5.S, D1.C, SJ4.2
- new net BUS_SCK_SCL: BUS-3.S, U1.IO38
- new net CAM_PWRDN: K1.17, U1.IO10
- new net IRLED_ON: Q2.G, U1.IO35
- new net LED_ON: R3.2, U1.IO5
- new net N$8: Q2.D, R2.2, R4.2, SJ5.1
- new net SD_CS0: R43.2, SDCARD.CD/DATA3, U1.IO17
- new net SD_MISO: R38.2, SDCARD.DATA0, U1.IO14
- new net SD_MOSI: R40.2, SDCARD.CMD, U1.IO16
- new net V: C3.1, D2.C, D3.C, IC1.VIN
- new net VEXT: D3.A, PAD5.P
- net CAM_D0: now also U1.IO13
- net CAM_D1: now also U1.IO4
- net CAM_D2: now also U1.IO34
- net CAM_D3: now also U1.IO37
- net CAM_D4: now also U1.IO12
- net CAM_D5: now also U1.IO26
- net CAM_D6: now also U1.IO21
- net CAM_D7: now also U1.IO18
- net CAM_HSYNC: now also U1.IO3
- net CAM_ON: now also U1.IO36
- net CAM_RESET: now also U1.IO11; no longer R19.2
- net CAM_SCL: now also PAD3.P, U1.IO7; no longer U1.IO5
- net CAM_SDA: now also PAD4.P, U1.IO8; no longer U1.IO4
- net CAM_U1.2: now also C22.1, IC3.VCC; no longer C21.2, IC11.VO
- net CAM_U2.8: now also C21.2, IC2.VCC; no longer C22.1, IC12.VO
- net CAM_XCLK: now also U1.IO1
- net ESP_EN: now also D1.A; no longer RESET.2
- net ESP_TDI: now also U1.IO41
- net GND: now also BOOT.1, BUS-6.S, IC1.GND, IC3.GND, LED1.C, LED2.C, LED_DBG.C, PAD1.P, PAD6.P; no longer BOOT.3, BOOT.4, C1.1, C5.1, C6.1, C7.1, C9.1, GPS-6.S, IC11.GND, IC12.GND, LED_B.C, R17.2, RESET.3, RESET.4, U2.GND, U3.GND
- net N$1: now also LED1.A, R4.1; no longer C6.2, Q3.2, U1.IO15
- net N$2: now also SJ4.1, U1.IO46; no longer C5.2, Q3.1, U1.IO14
- net N$3: now also LED2.A, R2.1; no longer C7.2, R3.1, USB.2
- net N$4: now also LED_DBG.A, R3.1; no longer C9.2, R4.1, USB.3
- net SD_CLK: now also U1.IO15
- net SD_ON: now also U1.IO6
- net U3.3: now also SJ1.1
- net USB_DM: now also U1.IO19, USB.2; no longer R3.2
- net USB_DP: now also U1.IO20, USB.3; no longer R4.2
- net USB_VBUS: now also D2.A
- net VCC: now also BUS-2.S, IC1.VCC, PAD2.P, Q2.S, SJ1.2, SJ3.1, SJ5.2; no longer C1.2, IC2.VO, R2.2, R5.2, U2.VCC, U3.VCC
- net VCC_CAM: now also IC2.VIN, IC3.VIN, SJ3.2; no longer IC11.VI, IC12.VI, R19.1
Other:
- note added: "(I2C/SPI BUS)"
- moved on the sheet: C10, C21, C22, C3, C8, H1, H2, Q1, R2, R3, R38, R39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
