File: hw/esp32buscam_01.brd (EAGLE design)
At the start: 33 x 19.1 mm, 51 parts, among them IC11 MCP1703DB, IC12 MCP1703DB, IC2 MCP1703DB, K1 68712414522, Q1 IRLML2244, Q4 IRLML2244, U1 ESP32-S2-MINI-1, U2 FLASH, U3 ESP-PSRAM64, X1 JTAG, X2 PROG

Commit message: first 100% layout
Parts:
- removed C1, C5, C6, C7, C9: (no value), rcl:C0603
- removed GPS: BUS, con-amp-micromatch:MICROMATCH-6SMD
- removed IC11, IC12: MCP1703DB, linear:SOT223
- removed LED_B: G, led:CHIPLED_0805
- removed Q3: (no value), crystal:TC26V
- removed R17, R19, R21, R5: (no value), rcl:R0603
- removed RESET: (no value), Ergaenzung:TASTER-9314_SMD
- removed U2: FLASH, esp32s2mini:SOC008_SPA
- removed U3: ESP-PSRAM64, esp32s2mini:SOC008_SPA
- added BUS: BUS, con-amp-micromatch:MICROMATCH-6SMD
- added D1, D2, D3: (no value), diode:MINIMELF
- added IC1, IC3: MCP1703SOT-89, bytewerk-vreg:SOT89
- added LED1, LED2: (no value), led:LED5MM
- added LED_DBG: G, led:CHIPLED_0805
- added PAD1, PAD2, PAD3, PAD4, PAD5, PAD6: (no value), wirepad:1,6/0,9
- added Q2: IRLML2244, User-Submitted:SOT23-3
- added SJ1, SJ3, SJ4, SJ5: (no value), jumper:SJ
- BOOT: device Ergaenzung:TASTER-9314_SMD -> jumper:SJ
- IC2: value MCP1703DB -> MCP1703SOT-89; device linear:SOT223 -> bytewerk-vreg:SOT89
- R2, R3, R4: device rcl:R0603 -> rcl:R0402
- moved C2 103.4 mm to (22.1, 4.06), turned to 270 degrees
- moved Q4 90.6 mm to (19.9, 17.8), flipped to the bottom
- moved R39 86.9 mm to (2.54, 1.27), flipped to the bottom, turned to 180 degrees
- moved C3 86.6 mm to (29.8, 11.9), turned to 90 degrees
- moved C17 85.9 mm to (10.2, 17.8), flipped to the bottom, turned to 90 degrees
- moved C8 81.7 mm to (9.14, 1.65)
- moved R38 80.9 mm to (2.54, 2.92), flipped to the bottom, turned to 180 degrees
- moved C10 80.3 mm to (13.1, 1.40)
- moved R20 80.0 mm to (15.9, 17.8), flipped to the bottom, turned to 270 degrees
- moved R1 80.0 mm to (16.8, 1.65), turned to 180 degrees
- moved R4 78.8 mm to (24.8, 18.9), flipped to the bottom
- moved R7 78.6 mm to (12.1, 17.8), flipped to the bottom, turned to 90 degrees
- moved R3 78.1 mm to (8.51, 3.43), turned to 180 degrees
- moved R6 77.3 mm to (14.0, 17.8), flipped to the bottom, turned to 90 degrees
- moved Q1 76.3 mm to (2.67, 12.1), flipped to the bottom, turned to 270 degrees
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Connections:
- removed net CAM_HREF: U1.7
- removed net CAM_PWDN: K1.17, R17.1
- removed net ESP_CS1: R2.1, U3.1
- removed net ESP_CS2: R5.1, U2.1
- removed net ESP_TDI(: U1.37
- removed net MTDO: R21.2
- removed net N$21: LED_B.A, R21.1
- removed net N$6: U1.5
- removed net SD_CMD: R40.2, SDCARD.3
- removed net SD_D0: R38.2, SDCARD.7
- removed net SD_D3: R43.2, SDCARD.2
- removed net SPICLK: U2.6, U3.6
- removed net SPID: U2.5, U3.5
- removed net SPIHD: U2.7, U3.7
- removed net SPIQ: U2.2, U3.2
- removed net SPIWP: U2.3, U3.3
- removed net SPI_MISO: GPS.1
- removed net SPI_MOSI: GPS.4
- removed net SPI_RESET: GPS.5
- removed net SPI_SCK: GPS.3
- removed net UBUS: GPS.2
- removed net USB_ID: USB.4
- removed net VBAT: C3.1, IC2.1
- new net BUS_MISO_INT: BUS.1, U1.41
- new net BUS_MOSI_SDA: BUS.4, U1.13
- new net BUS_RESET: BUS.5, D1.C, SJ4.2
- new net BUS_SCK_SCL: BUS.3, U1.34
- new net CAM_PWRDN: K1.17, U1.14
- new net IRLED_ON: Q2.1, U1.31
- new net LED_ON: R3.2, U1.9
- new net N$8: Q2.3, R2.2, R4.2, SJ5.1
- new net SD_CS0: R43.2, SDCARD.2, U1.21
- new net SD_MISO: R38.2, SDCARD.7, U1.18
- new net SD_MOSI: R40.2, SDCARD.3, U1.20
- new net V: C3.1, D2.C, D3.C, IC1.2, IC1.4
- new net VEXT: D3.A, PAD5.1
- net CAM_D0: now also U1.17
- net CAM_D1: now also U1.8
- net CAM_D2: now also U1.29
- net CAM_D3: now also U1.33
- net CAM_D4: now also U1.16
- net CAM_D5: now also U1.26
- net CAM_D6: now also U1.25
- net CAM_D7: now also U1.22
- net CAM_HSYNC: now also U1.7
- net CAM_ON: now also U1.32
- net CAM_RESET: now also U1.15; no longer R19.2
- net CAM_SCL: now also PAD3.1, U1.11; no longer U1.9
- net CAM_SDA: now also PAD4.1, U1.12; no longer U1.8
- net CAM_U1.2: now also C22.1, IC3.3; no longer C21.2, IC11.3
- net CAM_U2.8: now also C21.2, IC2.3; no longer C22.1, IC12.3
- net CAM_XCLK: now also U1.5
- net ESP_EN: now also D1.A; no longer RESET.2
- net ESP_TDI: now also U1.37
- net GND: now also BOOT.1, BUS.6, IC1.1, IC2.1, IC3.1, LED1.K, LED2.K, LED_DBG.C, PAD1.1, PAD6.1; no longer BOOT.3, BOOT.4, C1.1, C5.1, C6.1, C7.1, C9.1, GPS.6, IC11.2, IC12.2, IC2.2, LED_B.C, R17.2, RESET.3, RESET.4, U2.4, U3.4
- net N$1: now also LED1.A, R4.1; no longer C6.2, Q3.2, U1.19
- net N$2: now also SJ4.1, U1.44; no longer C5.2, Q3.1, U1.18
- net N$3: now also LED2.A, R2.1; no longer C7.2, R3.1, USB.2
- net N$4: now also LED_DBG.A, R3.1; no longer C9.2, R4.1, USB.3
- net SD_CLK: now also U1.19
- net SD_ON: now also U1.10
- net U3.3: now also SJ1.1
- net USB_DM: now also U1.23, USB.2; no longer R3.2
- net USB_DP: now also U1.24, USB.3; no longer R4.2
- net USB_VBUS: now also D2.A
- net VCC: now also BUS.2, IC1.3, PAD2.1, Q2.2, SJ1.2, SJ3.1, SJ5.2; no longer C1.2, IC2.3, R2.2, R5.2, U2.8, U3.8
- net VCC_CAM: now also IC2.2, IC2.4, IC3.2, IC3.4, SJ3.2; no longer IC11.1, IC12.1, R19.1
Routing:
- net GND: track 0.00 -> 168.2 mm, vias 0 -> 9
- net VCC: track 0.00 -> 75.8 mm, vias 0 -> 3
- net CAM_SDA: track 0.00 -> 37.1 mm, vias 0 -> 4
- net VCC_CAM: track 0.00 -> 35.8 mm, vias 0 -> 2
- net ESP_IO0: track 0.00 -> 34.0 mm, vias 0 -> 1
- net USB_DM: track 0.00 -> 28.7 mm, vias 0 -> 3
- net SD_MISO: track 0.00 -> 26.3 mm, vias 0 -> 2
- net BUS_RESET: track 0.00 -> 25.5 mm, vias 0 -> 4
- net USB_DP: track 0.00 -> 24.9 mm, vias 0 -> 1
- net CAM_SCL: track 0.00 -> 23.2 mm, vias 0 -> 3
- net SD_D2: track 0.00 -> 22.0 mm, vias 0 -> 1
- net SD_CS0: track 0.00 -> 21.1 mm, vias 0 -> 5
- net BUS_MOSI_SDA: track 0.00 -> 21.0 mm, vias 0 -> 5
- net SD_MOSI: track 0.00 -> 20.6 mm, vias 0 -> 2
- net SD_CLK: track 0.00 -> 20.2 mm, vias 0 -> 5
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Other:
- board size 33 x 19.1 mm -> 33.3 x 20.1 mm

Commit message: -
Parts:
- moved SJ5 0.57 mm to (22.6, 18.5)
- moved C21 0.57 mm to (9.27, 10.3)
- moved D2 0.57 mm to (27.2, 11.3)
- moved IC1 0.57 mm to (28.4, 12.3)
- moved R4 0.57 mm to (25.0, 19.4)
- moved SJ3 0.57 mm to (19.7, 18.5)
- moved Q1 0.57 mm to (2.92, 12.6)
- moved C10 0.57 mm to (13.3, 1.91)
- moved C2 0.57 mm to (22.4, 4.57)
- moved C22 0.57 mm to (13.7, 10.3)
- moved IC2 0.57 mm to (9.27, 7.24)
- moved PAD1 0.57 mm to (13.0, 3.68)
- moved PAD4 0.57 mm to (20.6, 3.68)
- moved SJ4 0.57 mm to (26.3, 1.91)
- moved USB 0.57 mm to (28.3, 1.91)
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Routing:
- net GND: vias 9 -> 22
- added copper zone on layer 1, net GND
- added copper zone on layer 16, net GND
Other:
- board size 33.3 x 20.1 mm -> 33.5 x 20.3 mm
