File: hw/esp32buscam_02.sch (EAGLE design)
At the start: 54 parts, among them IC1 MCP1703SOT-89, IC2 MCP1703SOT-89, IC3 MCP1703SOT-89, K1 68712414522, Q1 IRLML2244, Q2 IRLML2244, Q4 IRLML2244, U1 ESP32-S2-MINI-1, X1 JTAG, X2 PROG

Commit message: -
Parts:
- removed D3: (no value), diode:DIODE-MINIMELF
- removed H1, H2: MOUNT-HOLE2.8, holes:MOUNT-HOLE2.8
- removed LED_DBG: G, led:LEDCHIPLED_0805
- removed PAD1, PAD2, PAD3, PAD4, PAD5, PAD6: (no value), wirepad:1,6/0,9
- removed Q1: IRLML2244, User-Submitted:MOSFET-PCHANNELIRLML2244
- removed R3: (no value), rcl:R-EU_R0402
- removed R38, R39, R40, R41, R42, R43: 10k, rcl:R-EU_R0805
- removed SDCARD: 47309-3351, con-molex-microsd:47309-3351
- removed SJ1: (no value), jumper:SJ
- removed X1: JTAG, _hhn_con_pinhead_box_1mm27:PHB_1MM27_2X05_SNS
- removed X2: PROG, _hhn_con_pinhead_box_1mm27:PHB_1MM27_2X03_SNS
Connections:
- removed net N$4: LED_DBG.A, R3.1
- removed net SD_D1: R39.2, SDCARD.DATA1
- removed net SD_D2: R42.2, SDCARD.DATA2
- removed net U3.3: Q1.D, R38.1, R39.1, R40.1, R41.1, R42.1, R43.1, SDCARD.VDD, SJ1.1
- removed net VEXT: D3.A, PAD5.P
- net CAM_SCL: no longer PAD3.P
- net CAM_SDA: no longer PAD4.P
- net ESP_EN: no longer X2.1
- net ESP_IO0: no longer X2.6
- net ESP_RXD: no longer X2.5
- net ESP_TCK: no longer X1.4
- net ESP_TDI: no longer X1.8
- net ESP_TDO: no longer X1.6
- net ESP_TMS: no longer X1.2
- net ESP_TXD: no longer X2.3
- net GND: no longer LED_DBG.C, PAD1.P, PAD6.P, SDCARD.G1, SDCARD.G2, SDCARD.VSS, X1.3, X1.5, X1.7, X1.9, X2.4
- net LED_ON: no longer R3.2
- net SD_CLK: no longer R41.2, SDCARD.CLK
- net SD_CS0: no longer R43.2, SDCARD.CD/DATA3
- net SD_MISO: no longer R38.2, SDCARD.DATA0
- net SD_MOSI: no longer R40.2, SDCARD.CMD
- net SD_ON: no longer Q1.G
- net V: no longer D3.C
- net VCC: no longer PAD2.P, Q1.S, SJ1.2, X1.1, X2.2
